Commit message: Modify: URDF
modify camera location.

File: src/isaac_so_arm101/robots/piper_description/urdf/piper_description_with_d405.urdf (robot description, URDF)
Before this commit: robot piper_camera, 22 links, 21 joints
Links:
- link camera_bottom_screw_frame: mass None -> 0.001
- link camera_color_frame: mass None -> 0.001
- link camera_color_optical_frame: mass None -> 0.001
- link camera_depth_frame: mass None -> 0.001
- link camera_depth_optical_frame: mass None -> 0.001
- link camera_infra1_frame: mass None -> 0.001
- link camera_infra1_optical_frame: mass None -> 0.001
- link camera_infra2_frame: mass None -> 0.001
- link camera_infra2_optical_frame: mass None -> 0.001
Joints:
- joint camera_joint: origin xyz=-0.0425 0 0.038 rpy=0 -1.5707963267948966 0 -> xyz=-0.0425 0 0.055 rpy=0 -1.5707963267948966 0
